Commit message: Added docs and updated repository usage instructions.

File: src/roarm_main/roarm_description/urdf/bases/roarm_m2.xacro (robot description, xacro)
@@ -1,6 +1,10 @@
 <?xml version="1.0" ?>
 <robot name="roarm_m2" xmlns:xacro="http://www.ros.org/wiki/xacro">
+<xacro:macro name="add_depth_camera" params="add_depth_camera"></xacro:macro>
 <xacro:arg name="add_depth_camera" default="false"/>
 <xacro:property name="add_depth_camera" value="$(arg add_depth_camera)"/>
+<xacro:macro name="add_camera" params="add_camera"></xacro:macro>
+<xacro:arg name="add_camera" default="false"/>
+<xacro:property name="add_camera" value="$(arg add_camera)"/>
 <xacro:arg name="gripper_type" default="angular_gear"/>
 <xacro:property name="gripper_type" value="$(arg gripper_type)"/>
@@ -8,12 +12,37 @@
 <xacro:include filename="$(find roarm_description)/urdf/gazebo/roarm_m2.trans" />
 <xacro:include filename="$(find roarm_description)/urdf/gazebo/roarm_m2.gazebo" />
-<!-- <xacro:if value="${add_depth_camera}">
+<xacro:if value="${add_depth_camera}">
 <xacro:include filename="$(find roarm_description)/urdf/camera/depth_camera.xacro" />
 <xacro:include filename="$(find roarm_description)/urdf/camera/depth_camera.gazebo.xacro" />
+<!-- <xacro:oak use_gazebo="true">
+  <parent link="link4" />
+  <origin xyz="-0.066257 -0.0523 0" rpy="1.5708 0 -1.5708" />
+  oak cam in hand
+</xacro:oak>   -->
 <xacro:oak use_gazebo="true">
-  <parent link="link3" />
-  <origin xyz="-0.06 -0.2 0" rpy="1.5708 0 -1.5708" />
+  <parent link="base_link" />
+  <origin xyz="0.06531 0 0.021953" rpy="0 0 0" />
+  <!-- usb cam out hand -->
 </xacro:oak>
-</xacro:if> -->
+</xacro:if>
+<xacro:if value="${add_camera}">
+<xacro:include filename="$(find roarm_description)/urdf/camera/camera.xacro" />
+<xacro:include filename="$(find roarm_description)/urdf/camera/camera.gazebo.xacro" />
+<xacro:cam use_gazebo="true">
+  <xacro:if value="${gripper_type == 'angular_direct'}">
+    <parent link="link3" />
+    <origin xyz="-0.062588 -0.181612 0" rpy="1.5708 0 -1.3963" />
+  </xacro:if>
+  <xacro:if value="${gripper_type == 'angular_gear'}">
+    <parent link="link3" />
+    <!-- <origin xyz="-0.046 -0.183536 0" rpy="1.5708 0 -1.5708" /> -->
+    <origin xyz="-0.020898 -0.239246 0" rpy="1.5708 0 -1.5708" />
+    <!-- usb cam in hand -->
+  </xacro:if>
+    <!-- <parent link="base_link" />
+    <origin xyz="0.06531 0 0.021953" rpy="0 0 0" /> -->
+    <!-- usb cam out hand -->
+  </xacro:cam>
+</xacro:if>
 <link name="world"></link>
 <link name="base_link">
@@ -123,5 +152,5 @@
   <child  link="link3" />
   <axis xyz="0 0 1" />
-  <limit lower="-1" upper="2.95" effort="0" velocity="0" />
+  <limit lower="0" upper="2.95" effort="0" velocity="0" />
 </joint>
 <xacro:if value="${gripper_type == 'angular_direct'}">

File: src/roarm_main/roarm_description/urdf/bases/roarm_m3.xacro (robot description, xacro)
@@ -1,22 +1,45 @@
 <?xml version="1.0" ?>
 <robot name="roarm_m3" xmlns:xacro="http://www.ros.org/wiki/xacro">
+<xacro:include filename="$(find roarm_description)/urdf/materials.xacro" />
+<xacro:include filename="$(find roarm_description)/urdf/gazebo/roarm_m3.trans" />
+<xacro:include filename="$(find roarm_description)/urdf/gazebo/roarm_m3.gazebo" />
 <xacro:macro name="add_depth_camera" params="add_depth_camera"></xacro:macro>
 <xacro:arg name="add_depth_camera" default="false"/>
 <xacro:property name="add_depth_camera" value="$(arg add_depth_camera)"/>
-<xacro:include filename="$(find roarm_description)/urdf/materials.xacro" />
-<xacro:include filename="$(find roarm_description)/urdf/gazebo/roarm_m3.trans" />
-<xacro:include filename="$(find roarm_description)/urdf/gazebo/roarm_m3.gazebo" />
+<xacro:macro name="add_camera" params="add_camera"></xacro:macro>
+<xacro:arg name="add_camera" default="false"/>
+<xacro:property name="add_camera" value="$(arg add_camera)"/>
 <xacro:if value="${add_depth_camera}">
 <xacro:include filename="$(find roarm_description)/urdf/camera/depth_camera.xacro" />
 <xacro:include filename="$(find roarm_description)/urdf/camera/depth_camera.gazebo.xacro" />
-<xacro:oak use_gazebo="true">
+<!-- <xacro:oak use_gazebo="true">
   <parent link="link4" />
   <origin xyz="-0.066257 -0.0523 0" rpy="1.5708 0 -1.5708" />
+  oak cam in hand
+</xacro:oak>   -->
+<xacro:oak use_gazebo="true">
+  <parent link="base_link" />
+  <origin xyz="0.06531 0 0.021953" rpy="0 0 0" />
+  <!-- usb cam out hand -->
 </xacro:oak>
+</xacro:if>
+<xacro:if value="${add_camera}">
+<xacro:include filename="$(find roarm_description)/urdf/camera/camera.xacro" />
+<xacro:include filename="$(find roarm_description)/urdf/camera/camera.gazebo.xacro" />
+<xacro:cam use_gazebo="true">
+  <parent link="link4" />
+  <origin xyz="-0.046 -0.072938 0" rpy="1.5708 0 -1.3963" />
+  <!-- usb cam in hand -->
+</xacro:cam>
+<!-- <xacro:cam use_gazebo="true">
+  <parent link="base_link" />
+  <origin xyz="0.06531 0 0.021953" rpy="0 0 0" />
+  usb cam out hand
+</xacro:cam>  -->
 </xacro:if>
 <link name="world"></link>
 <link name="base_link">
   <inertial>
-    <origin xyz="-0.0068 0 -0.03" rpy="0 0 0" />
+    <origin xyz="0.0032 0 0.0417" rpy="0 0 0" />
     <mass value="0.2562183" />
     <inertia ixx="0.00029211" ixy="0" ixz="0" iyy="0.00035719" iyz="0" izz="0.000349421" />
@@ -158,5 +181,5 @@
 <link name="hand_tcp"></link>
 <joint name="world_to_base_link" type="fixed">
-  <origin xyz="0.0 0.0 0.0701" rpy="0 0 0"/>
+  <origin xyz="0.0 0.0 0.0" rpy="0 0 0"/>
   <parent link="world"/>
   <child link="base_link"/>
@@ -164,5 +187,5 @@
 </joint>
 <joint name="base_link_to_link1" type="revolute">
-  <origin xyz="0.0 0.0 0.0" rpy="0 0 0"/>
+  <origin xyz="0.0100000008759151 0.0 0.0716" rpy="0 0 0"/>
   <parent link="base_link"/>
   <child link="link1"/>
@@ -191,5 +214,5 @@
   <axis xyz="0.0 0.0 1.0"/>
   <limit
-    lower="-1"
+    lower="0"
     upper="2.95"
     effort="0"

File: src/roarm_main/roarm_moveit/config/roarm_m2/roarm_m2.ros2_control.xacro (robot description, xacro)
@@ -1,5 +1,5 @@
 <?xml version="1.0"?>
 <robot xmlns:xacro="http://www.ros.org/wiki/xacro">
-    <xacro:macro name="roarm_m2_ros2_control" params="use_gazebo GZ_VERSION initial_positions_file">
+    <xacro:macro name="roarm_m2_ros2_control" params="use_gazebo GZ_VERSION gripper_type initial_positions_file">
         <xacro:property name="initial_positions" value="${load_yaml(initial_positions_file)['initial_positions']}"/>
         <ros2_control name="RoarmHardware" type="system">
@@ -45,4 +45,5 @@
                 <state_interface name="velocity"/>
             </joint>
+            <xacro:if value="${gripper_type == 'angular_gear'}">
             <joint name="gripper_left_joint1">
               <param name="mimic">gripper_joint</param>
@@ -99,4 +100,5 @@
               <state_interface name="velocity"/>
             </joint>
+            </xacro:if>
         </ros2_control>
     </xacro:macro>

File: src/roarm_main/roarm_moveit/config/roarm_m2/roarm_m2.urdf.xacro (robot description, xacro)
@@ -7,9 +7,12 @@
 <xacro:arg name="GZ_VERSION" default="classic"/>
 <xacro:property name="GZ_VERSION" value="$(arg GZ_VERSION)"/>
+<xacro:macro name="gripper_type" params="gripper_type"></xacro:macro>
+<xacro:arg name="gripper_type" default="angular_gear"/>
+<xacro:property name="gripper_type" value="$(arg gripper_type)"/>
 <xacro:arg name="initial_positions_file" default="initial_positions.yaml" />
 <!-- Import roarm urdf file -->
 <xacro:include filename="$(find roarm_description)/urdf/bases/roarm_m2.xacro" />
 <xacro:include filename="roarm_m2.ros2_control.xacro" />
-<xacro:roarm_m2_ros2_control use_gazebo="$(arg use_gazebo)" GZ_VERSION="$(arg GZ_VERSION)" initial_positions_file="$(arg initial_positions_file)"/>
+<xacro:roarm_m2_ros2_control use_gazebo="$(arg use_gazebo)" GZ_VERSION="$(arg GZ_VERSION)" gripper_type="$(arg gripper_type)" initial_positions_file="$(arg initial_positions_file)"/>
 <gazebo>
     <xacro:if value="${GZ_VERSION == 'classic'}">

Commit message: Compatible with the new version of Gazebo.

File: src/roarm_main/roarm_description/urdf/bases/roarm_m2.xacro (robot description, xacro)
@@ -138,5 +138,5 @@
   <child link="link1" />
   <axis xyz="0 0 1" />
-  <limit lower="-3.1416" upper="3.1416" effort="0" velocity="0" />
+  <limit lower="-3.1416" upper="3.1416" effort="20" velocity="3.14" />
 </joint>
 <joint name="link1_to_link2" type="revolute">
@@ -145,5 +145,5 @@
   <child link="link2" />
   <axis xyz="0 0 1" />
-  <limit lower="-1.5708" upper="1.5708" effort="0" velocity="0" />
+  <limit lower="-1.5708" upper="1.5708" effort="20" velocity="3.14" />
 </joint>
 <joint name="link2_to_link3" type="revolute">
@@ -152,5 +152,5 @@
   <child  link="link3" />
   <axis xyz="0 0 1" />
-  <limit lower="0" upper="2.95" effort="0" velocity="0" />
+  <limit lower="0" upper="2.95" effort="20" velocity="3.14" />
 </joint>
 <xacro:if value="${gripper_type == 'angular_direct'}">

File: src/roarm_main/roarm_description/urdf/bases/roarm_m3.xacro (robot description, xacro)
@@ -194,6 +194,6 @@
     lower="-3.1416"
     upper="3.1416"
-    effort="0"
-    velocity="0" />
+    effort="20"
+    velocity="3.14" />
 </joint>
 <joint name="link1_to_link2" type="revolute">
@@ -205,6 +205,6 @@
     lower="-1.5708"
     upper="1.5708"
-    effort="0"
-    velocity="0" />
+    effort="20"
+    velocity="3.14" />
 </joint>
 <joint name="link2_to_link3" type="revolute">
@@ -216,6 +216,6 @@
     lower="0"
     upper="2.95"
-    effort="0"
-    velocity="0" />
+    effort="20"
+    velocity="3.14" />
 </joint>
 <joint name="link3_to_link4" type="revolute">
@@ -227,6 +227,6 @@
     lower="-1.5708"
     upper="1.5708"
-    effort="0"
-    velocity="0" />
+    effort="20"
+    velocity="3.14" />
 </joint>
 <joint name="link4_to_link5" type="revolute">
@@ -238,6 +238,6 @@
     lower="-3.1416"
     upper="3.1416"
-    effort="0"
-    velocity="0" />
+    effort="20"
+    velocity="3.14" />
 </joint>
 <joint name="link5_to_gripper_link" type="revolute">
@@ -249,6 +249,6 @@
     lower="0"
     upper="1.5"
-    effort="0"
-    velocity="0" />
+    effort="20"
+    velocity="3.14" />
 </joint>
 <joint name="link5_to_hand_tcp" type="fixed">

File: src/roarm_main/roarm_description/urdf/gripper/gripper.xacro (robot description, xacro)
@@ -43,5 +43,5 @@
   <joint name="gripper_joint" type="revolute">
     <axis xyz="0 0 -1"/>
-    <limit effort="1000.0" lower="0" upper="1.57" velocity="0.5"/>
+    <limit effort="20.0" lower="0" upper="1.57" velocity="3.14"/>
     <parent link="gripper_base"/>
     <child link="gripper_link"/>

File: src/roarm_main/roarm_description/urdf/gripper/gripper_a.xacro (robot description, xacro)
@@ -163,5 +163,5 @@
   <joint name="gripper_joint" type="revolute">
     <axis xyz="0 0 -1"/>
-    <limit effort="1000.0" lower="0" upper="1.57" velocity="0.5"/>
+    <limit effort="20.0" lower="0" upper="1.57" velocity="3.14"/>
     <parent link="gripper_base"/>
     <child link="gripper_link"/>
@@ -170,5 +170,5 @@
   <joint name="gripper_left_joint1" type="revolute">
     <axis xyz="0 0 1"/>
-    <limit effort="1000.0" lower="-1.57" upper="1.57" velocity="0.5"/>
+    <limit effort="20.0" lower="-1.57" upper="1.57" velocity="3.14"/>
     <parent link="gripper_base"/>
     <child link="gripper_left1"/>
@@ -178,5 +178,5 @@
   <joint name="gripper_left_joint2" type="revolute">
     <axis xyz="0 0 1"/>
-    <limit effort="1000.0" lower="-1.57" upper="1.57" velocity="0.5"/>
+    <limit effort="20.0" lower="-1.57" upper="1.57" velocity="3.14"/>
     <parent link="gripper_base"/>
     <child link="gripper_left2"/>
@@ -186,5 +186,5 @@
   <joint name="gripper_left_joint3" type="revolute">
     <axis xyz="0 0 1"/>
-    <limit effort="1000.0" lower="-1.57" upper="1.57" velocity="0.5"/>
+    <limit effort="20.0" lower="-1.57" upper="1.57" velocity="3.14"/>
     <parent link="gripper_left2"/>
     <child link="gripper_left3"/>
@@ -194,5 +194,5 @@
   <joint name="gripper_right_joint1" type="revolute">
     <axis xyz="0 0 -1"/>
-    <limit effort="1000.0" lower="-1.57" upper="1.57" velocity="0.5"/>
+    <limit effort="20.0" lower="-1.57" upper="1.57" velocity="3.14"/>
     <parent link="gripper_base"/>
     <child link="gripper_right1"/>
@@ -202,5 +202,5 @@
   <joint name="gripper_right_joint2" type="revolute">
     <axis xyz="0 0 1"/>
-    <limit effort="1000.0" lower="-1.57" upper="1.57" velocity="0.5"/>
+    <limit effort="20.0" lower="-1.57" upper="1.57" velocity="3.14"/>
     <parent link="gripper_base"/>
     <child link="gripper_right2"/>
@@ -210,5 +210,5 @@
   <joint name="gripper_right_joint3" type="revolute">
     <axis xyz="0 0 1"/>
-    <limit effort="1000.0" lower="-1.57" upper="1.57" velocity="0.5"/>
+    <limit effort="20.0" lower="-1.57" upper="1.57" velocity="3.14"/>
     <parent link="gripper_right2"/>
     <child link="gripper_right3"/>
