Commit message: MTC core: Removed hardcoded base_link inverse transforms; restored upstream Humble planning-frame math (move_relative / compute_ik); removed cartesian_path debug prints Cameras: Meshes now use in-repo roarm_description (no ugv_description dependency); Harmonic camera topics aligned with the bridge (cam/image, hand_oak); /joint_states no longer bridged from GZ (comes from joint_state_broadcaster) Launch: command_control and MTC demo correctly forward use_rviz, add_camera, add_depth_camera MoveIt: Hand-eye collision pairs for M2/M3; YOLO pick-place uses arm_home_pose (M2 has no observe) Vision: Default base_frame is base_link (UGV setups must pass ugv_roarm_base_link) Docs: Gazebo / Vision / Cmd / MTC / Description aligned with the above

File: src/roarm_main/roarm_description/urdf/bases/roarm_m2.xacro (robot description, xacro)
@@ -1,10 +1,11 @@
 <?xml version="1.0" ?>
 <robot name="roarm_m2" xmlns:xacro="http://www.ros.org/wiki/xacro">
-<xacro:macro name="add_depth_camera" params="add_depth_camera"></xacro:macro>
+<!-- Declared here: this file is also an entry for roarm_description/display.launch.py -->
 <xacro:arg name="add_depth_camera" default="false"/>
-<xacro:property name="add_depth_camera" value="$(arg add_depth_camera)"/>
-<xacro:macro name="add_camera" params="add_camera"></xacro:macro>
+<!-- M2 depth-camera mount not designed yet; arg kept for launch compatibility. -->
 <xacro:arg name="add_camera" default="false"/>
 <xacro:property name="add_camera" value="$(arg add_camera)"/>
+<xacro:arg name="GZ_VERSION" default="classic"/>
+<xacro:property name="GZ_VERSION" value="$(arg GZ_VERSION)"/>
 <xacro:arg name="gripper_type" default="angular_gear"/>
 <xacro:property name="gripper_type" value="$(arg gripper_type)"/>
@@ -12,18 +13,4 @@
 <xacro:include filename="$(find roarm_description)/urdf/gazebo/roarm_m2.trans" />
 <xacro:include filename="$(find roarm_description)/urdf/gazebo/roarm_m2.gazebo" />
-<xacro:if value="${add_depth_camera}">
-<xacro:include filename="$(find roarm_description)/urdf/camera/depth_camera.xacro" />
-<xacro:include filename="$(find roarm_description)/urdf/camera/depth_camera.gazebo.xacro" />
-<!-- <xacro:oak use_gazebo="true">
-  <parent link="link4" />
-  <origin xyz="-0.066257 -0.0523 0" rpy="1.5708 0 -1.5708" />
-  oak cam in hand
-</xacro:oak>   -->
-<xacro:oak use_gazebo="true">
-  <parent link="base_link" />
-  <origin xyz="0.06531 0 0.021953" rpy="0 0 0" />
-  <!-- usb cam out hand -->
-</xacro:oak>
-</xacro:if>
 <xacro:if value="${add_camera}">
 <xacro:include filename="$(find roarm_description)/urdf/camera/camera.xacro" />

File: src/roarm_main/roarm_description/urdf/bases/roarm_m3.xacro (robot description, xacro)
@@ -4,22 +4,18 @@
 <xacro:include filename="$(find roarm_description)/urdf/gazebo/roarm_m3.trans" />
 <xacro:include filename="$(find roarm_description)/urdf/gazebo/roarm_m3.gazebo" />
-<xacro:macro name="add_depth_camera" params="add_depth_camera"></xacro:macro>
+<!-- Declared here: this file is also an entry for roarm_description/display.launch.py -->
 <xacro:arg name="add_depth_camera" default="false"/>
 <xacro:property name="add_depth_camera" value="$(arg add_depth_camera)"/>
-<xacro:macro name="add_camera" params="add_camera"></xacro:macro>
 <xacro:arg name="add_camera" default="false"/>
 <xacro:property name="add_camera" value="$(arg add_camera)"/>
+<xacro:arg name="GZ_VERSION" default="classic"/>
+<xacro:property name="GZ_VERSION" value="$(arg GZ_VERSION)"/>
 <xacro:if value="${add_depth_camera}">
 <xacro:include filename="$(find roarm_description)/urdf/camera/depth_camera.xacro" />
 <xacro:include filename="$(find roarm_description)/urdf/camera/depth_camera.gazebo.xacro" />
-<!-- <xacro:oak use_gazebo="true">
+<xacro:oak use_gazebo="true">
   <parent link="link4" />
   <origin xyz="-0.066257 -0.0523 0" rpy="1.5708 0 -1.5708" />
-  oak cam in hand
-</xacro:oak>   -->
-<xacro:oak use_gazebo="true">
-  <parent link="base_link" />
-  <origin xyz="0.06531 0 0.021953" rpy="0 0 0" />
-  <!-- usb cam out hand -->
+  <!-- oak cam in hand -->
 </xacro:oak>
 </xacro:if>

File: src/roarm_main/roarm_description/urdf/camera/camera.gazebo.xacro (robot description, xacro)
@@ -1,4 +1,7 @@
 <?xml version="1.0"?>
 <robot xmlns:xacro="http://ros.org/wiki/xacro">
+<!-- GZ_VERSION comes from the entry urdf.xacro (ugv_roarm / roarm_moveit). -->
+<!-- Gazebo Classic -->
+<xacro:if value="${GZ_VERSION == 'classic'}">
 <gazebo reference="cam_base_hand">
   <sensor name="cam" type="camera">
@@ -11,5 +14,5 @@
         <width>640</width>
         <height>480</height>
-        <format>RGB8</format>
+        <format>R8G8B8</format>
       </image>
       <clip>
@@ -32,3 +35,33 @@
   </sensor>
 </gazebo>
+</xacro:if>
+<!-- Gazebo Harmonic (images via ros_gz_bridge) -->
+<xacro:if value="${GZ_VERSION == 'harmonic'}">
+<gazebo reference="cam_base_hand">
+  <sensor name="cam" type="camera">
+    <gz_frame_id>camera_link</gz_frame_id>
+    <topic>cam/image</topic>
+    <always_on>true</always_on>
+    <visualize>true</visualize>
+    <update_rate>30</update_rate>
+    <camera name="cam">
+      <horizontal_fov>1.2</horizontal_fov>
+      <image>
+        <width>640</width>
+        <height>480</height>
+        <format>R8G8B8</format>
+      </image>
+      <clip>
+        <near>0.02</near>
+        <far>8</far>
+      </clip>
+      <noise>
+        <type>gaussian</type>
+        <mean>0.0</mean>
+        <stddev>0.007</stddev>
+      </noise>
+    </camera>
+  </sensor>
+</gazebo>
+</xacro:if>
 </robot>

File: src/roarm_main/roarm_description/urdf/camera/camera.xacro (robot description, xacro)
@@ -12,5 +12,5 @@
     <origin xyz="0 0 0" rpy="0 0 0" />
     <geometry>
-      <mesh filename="file://$(find ugv_description)/meshes/sensors/pt/pt_camera_link.stl" />
+      <mesh filename="file://$(find roarm_description)/meshes/camera/pt_camera_link.stl" />
     </geometry>
     <material name="silver"/>
@@ -19,5 +19,5 @@
     <origin xyz="0 0 0" rpy="0 0 0" />
     <geometry>
-      <mesh filename="file://$(find ugv_description)/meshes/sensors/pt/pt_camera_link.stl" />
+      <mesh filename="file://$(find roarm_description)/meshes/camera/pt_camera_link.stl" />
     </geometry>
   </collision>
@@ -47,5 +47,5 @@
     <origin xyz="0 0 0" rpy="0 0 0" />
     <geometry>
-      <mesh filename="file://$(find ugv_description)/meshes/sensors/pt/pt_camera_link.stl" />
+      <mesh filename="file://$(find roarm_description)/meshes/camera/pt_camera_link.stl" />
     </geometry>
     <material name="silver"/>
@@ -54,5 +54,5 @@
     <origin xyz="0 0 0" rpy="0 0 0" />
     <geometry>
-      <mesh filename="file://$(find ugv_description)/meshes/sensors/pt/pt_camera_link.stl" />
+      <mesh filename="file://$(find roarm_description)/meshes/camera/pt_camera_link.stl" />
     </geometry>
   </collision>

File: src/roarm_main/roarm_description/urdf/camera/depth_camera.gazebo.xacro (robot description, xacro)
@@ -1,4 +1,7 @@
 <?xml version="1.0"?>
 <robot xmlns:xacro="http://ros.org/wiki/xacro">
+<!-- GZ_VERSION comes from the entry urdf.xacro (ugv_roarm / roarm_moveit). -->
+<!-- Gazebo Classic -->
+<xacro:if value="${GZ_VERSION == 'classic'}">
 <gazebo reference="oak_base_hand">
   <sensor name="oak" type="depth">
@@ -11,5 +14,5 @@
         <width>640</width>
         <height>480</height>
-        <format>RGB8</format>
+        <format>R8G8B8</format>
       </image>
       <clip>
@@ -32,3 +35,33 @@
   </sensor>
 </gazebo>
+</xacro:if>
+<!-- Gazebo Harmonic (images via ros_gz_bridge) -->
+<xacro:if value="${GZ_VERSION == 'harmonic'}">
+<gazebo reference="oak_base_hand">
+  <sensor name="hand_oak" type="rgbd_camera">
+    <gz_frame_id>depth_camera_link</gz_frame_id>
+    <topic>hand_oak</topic>
+    <update_rate>30</update_rate>
+    <always_on>true</always_on>
+    <visualize>true</visualize>
+    <camera>
+      <horizontal_fov>1.2</horizontal_fov>
+      <image>
+        <width>640</width>
+        <height>480</height>
+      </image>
+      <clip>
+        <near>0.02</near>
+        <far>8.0</far>
+      </clip>
+      <depth_camera>
+        <clip>
+          <near>0.02</near>
+          <far>8.0</far>
+        </clip>
+      </depth_camera>
+    </camera>
+  </sensor>
+</gazebo>
+</xacro:if>
 </robot>

File: src/roarm_main/roarm_description/urdf/camera/depth_camera.xacro (robot description, xacro)
@@ -12,5 +12,5 @@
     <origin xyz="0 0 0" rpy="0 0 0" />
     <geometry>
-      <mesh filename="file://$(find ugv_description)/meshes/sensors/3d_camera_link.stl" />
+      <mesh filename="file://$(find roarm_description)/meshes/camera/3d_camera_link.stl" />
     </geometry>
     <material name="silver"/>
@@ -19,5 +19,5 @@
     <origin xyz="0 0 0" rpy="0 0 0" />
     <geometry>
-      <mesh filename="file://$(find ugv_description)/meshes/sensors/3d_camera_link.stl" />
+      <mesh filename="file://$(find roarm_description)/meshes/camera/3d_camera_link.stl" />
     </geometry>
   </collision>
@@ -47,5 +47,5 @@
     <origin xyz="0 0 0" rpy="0 0 0" />
     <geometry>
-      <mesh filename="file://$(find ugv_description)/meshes/sensors/3d_camera_link.stl" />
+      <mesh filename="file://$(find roarm_description)/meshes/camera/3d_camera_link.stl" />
     </geometry>
     <material name="silver"/>
@@ -54,5 +54,5 @@
     <origin xyz="0 0 0" rpy="0 0 0" />
     <geometry>
-      <mesh filename="file://$(find ugv_description)/meshes/sensors/3d_camera_link.stl" />
+      <mesh filename="file://$(find roarm_description)/meshes/camera/3d_camera_link.stl" />
     </geometry>
   </collision>

File: src/roarm_main/roarm_moveit/config/roarm_m2/roarm_m2.urdf.xacro (robot description, xacro)
@@ -1,4 +1,5 @@
 <?xml version="1.0"?>
 <robot xmlns:xacro="http://www.ros.org/wiki/xacro" name="roarm_m2">
+<!-- Single entry-point declarations for standalone RoArm M2. -->
 <xacro:macro name="use_gazebo" params="use_gazebo"></xacro:macro>
 <xacro:arg name="use_gazebo" default="false"/>
@@ -10,4 +11,10 @@
 <xacro:arg name="gripper_type" default="angular_gear"/>
 <xacro:property name="gripper_type" value="$(arg gripper_type)"/>
+<xacro:macro name="add_camera" params="add_camera"></xacro:macro>
+<xacro:arg name="add_camera" default="false"/>
+<xacro:property name="add_camera" value="$(arg add_camera)"/>
+<xacro:macro name="add_depth_camera" params="add_depth_camera"></xacro:macro>
+<xacro:arg name="add_depth_camera" default="false"/>
+<xacro:property name="add_depth_camera" value="$(arg add_depth_camera)"/>
 <xacro:arg name="initial_positions_file" default="initial_positions.yaml" />
 <!-- Import roarm urdf file -->
@@ -25,4 +32,7 @@
         <parameters>$(find roarm_moveit)/config/roarm_m2/ros2_controllers.yaml</parameters>
     </plugin>
+    <plugin filename="gz-sim-sensors-system" name="gz::sim::systems::Sensors">
+        <render_engine>ogre2</render_engine>
+    </plugin>
     </xacro:if>
 </gazebo>

File: src/roarm_main/roarm_moveit/config/roarm_m3/roarm_m3.urdf.xacro (robot description, xacro)
@@ -1,4 +1,5 @@
 <?xml version="1.0"?>
 <robot xmlns:xacro="http://www.ros.org/wiki/xacro" name="roarm_m3">
+<!-- Single entry-point declarations for standalone RoArm M3. -->
 <xacro:macro name="use_gazebo" params="use_gazebo"></xacro:macro>
 <xacro:arg name="use_gazebo" default="false"/>
@@ -7,8 +8,11 @@
 <xacro:arg name="GZ_VERSION" default="classic"/>
 <xacro:property name="GZ_VERSION" value="$(arg GZ_VERSION)"/>
+<xacro:macro name="add_camera" params="add_camera"></xacro:macro>
+<xacro:arg name="add_camera" default="false"/>
+<xacro:property name="add_camera" value="$(arg add_camera)"/>
+<xacro:macro name="add_depth_camera" params="add_depth_camera"></xacro:macro>
 <xacro:arg name="add_depth_camera" default="false"/>
 <xacro:property name="add_depth_camera" value="$(arg add_depth_camera)"/>
 <xacro:include filename="$(find roarm_description)/urdf/bases/roarm_m3.xacro" />
-<xacro:add_depth_camera add_depth_camera="$(arg add_depth_camera)"/>
 <xacro:arg name="initial_positions_file" default="initial_positions.yaml" />
 <xacro:include filename="roarm_m3.ros2_control.xacro" />
@@ -24,4 +28,7 @@
         <parameters>$(find roarm_moveit)/config/roarm_m3/ros2_controllers.yaml</parameters>
     </plugin>
+    <plugin filename="gz-sim-sensors-system" name="gz::sim::systems::Sensors">
+        <render_engine>ogre2</render_engine>
+    </plugin>
     </xacro:if>
 </gazebo>
